Commit message: add robot action testing

File: mechlmm_ws/src/turtlebot3_manipulation/turtlebot3_manipulation_description/urdf/turtlebot3_waffle_pi.urdf.xacro (robot description, xacro)
@@ -170,5 +170,5 @@
     <parent link="${prefix}base_link"/>
     <child link="${prefix}camera_link"/>
-    <origin xyz="-0.4 -0.011 1" rpy="0 0.8 0"/>
+    <origin xyz="-0.3 0.3 0.6" rpy="0 0.6 -0.3"/>
   </joint>
   <link name="${prefix}camera_link">
