Commit message: remove collision of head camera

File: mechlmm_noetic_ws/src/turtlebot3_manipulation/turtlebot3_manipulation_description/urdf/turtlebot3_manipulation_robot.urdf.xacro (robot description, xacro)
@@ -12,14 +12,4 @@
   </joint>
   <link name="head_camera_link">
-    <inertial>
-      <mass value="0.1"/>
-      <origin xyz="0 0 0"/>
-      <inertia ixx="0.01" iyy="0.01" izz="0.01" ixy="0" ixz="0" iyz="0"/>
-    </inertial>
-    <collision>
-      <geometry>
-        <box size="0.05 0.05 0.05"/>
-      </geometry>
-    </collision>
     <visual>
       <geometry>
