Commit message: update simulation environment

File: mechlmm_noetic_ws/src/turtlebot3_manipulation/turtlebot3_manipulation_description/urdf/open_manipulator_x.gazebo.xacro (robot description, xacro)
@@ -49,3 +49,76 @@
     </plugin>
   </gazebo>
+  <!-- camera -->
+  <gazebo reference="hand_camera_link">
+    <sensor type="camera" name="camera1">
+      <update_rate>30.0</update_rate>
+      <camera name="hand">
+        <horizontal_fov>1.3962634</horizontal_fov>
+        <image>
+          <width>640</width>
+          <height>360</height>
+          <format>R8G8B8</format>
+        </image>
+        <clip>
+          <near>0.02</near>
+          <far>300</far>
+        </clip>
+        <noise>
+          <type>gaussian</type>
+          <mean>0.0</mean>
+          <stddev>0.007</stddev>
+        </noise>
+      </camera>
+      <plugin name="camera_controller" filename="libgazebo_ros_camera.so">
+        <alwaysOn>true</alwaysOn>
+        <updateRate>0.0</updateRate>
+        <cameraName>camera/hand</cameraName>
+        <imageTopicName>image_raw</imageTopicName>
+        <cameraInfoTopicName>camera_info</cameraInfoTopicName>
+        <frameName>hand_camera_link</frameName>
+        <hackBaseline>0.07</hackBaseline>
+        <distortionK1>0.0</distortionK1>
+        <distortionK2>0.0</distortionK2>
+        <distortionK3>0.0</distortionK3>
+        <distortionT1>0.0</distortionT1>
+        <distortionT2>0.0</distortionT2>
+      </plugin>
+    </sensor>
+  </gazebo>
+  <gazebo reference="head_camera_link">
+    <sensor type="camera" name="camera1">
+      <update_rate>30.0</update_rate>
+      <camera name="head">
+        <horizontal_fov>1.3962634</horizontal_fov>
+        <image>
+          <width>640</width>
+          <height>360</height>
+          <format>R8G8B8</format>
+        </image>
+        <clip>
+          <near>0.02</near>
+          <far>300</far>
+        </clip>
+        <noise>
+          <type>gaussian</type>
+          <mean>0.0</mean>
+          <stddev>0.007</stddev>
+        </noise>
+      </camera>
+      <plugin name="camera_controller" filename="libgazebo_ros_camera.so">
+        <alwaysOn>true</alwaysOn>
+        <updateRate>0.0</updateRate>
+        <cameraName>camera/head</cameraName>
+        <imageTopicName>image_raw</imageTopicName>
+        <cameraInfoTopicName>camera_info</cameraInfoTopicName>
+        <frameName>head_camera_link</frameName>
+        <hackBaseline>0.07</hackBaseline>
+        <distortionK1>0.0</distortionK1>
+        <distortionK2>0.0</distortionK2>
+        <distortionK3>0.0</distortionK3>
+        <distortionT1>0.0</distortionT1>
+        <distortionT2>0.0</distortionT2>
+      </plugin>
+    </sensor>
+  </gazebo>
 </robot>

File: mechlmm_noetic_ws/src/turtlebot3_manipulation/turtlebot3_manipulation_description/urdf/open_manipulator_x.urdf.xacro (robot description, xacro)
@@ -242,3 +242,21 @@
     </inertial>
   </link>
+  <link name="hand_camera_link">
+    <!-- <visual>
+      <origin xyz="0 0 0" rpy="0 0 0"/>
+      <geometry>
+        <box size="0.01 0.01 0.01" />
+      </geometry>
+    </visual> -->
+    <inertial>
+      <mass value="0.1"/>
+      <origin xyz="0 0 0"/>
+      <inertia ixx="0.01" iyy="0.01" izz="0.01" ixy="0" ixz="0" iyz="0"/>
+    </inertial>
+  </link>
+  <joint name="hand_camera_base_fixed" type="fixed">
+    <origin xyz="0.0 0.0 0.0" rpy="0.0 0.0 0.0"/>
+    <parent link="end_effector_link"/>
+    <child link="hand_camera_link"/>
+  </joint>
 </robot>

File: mechlmm_noetic_ws/src/turtlebot3_manipulation/turtlebot3_manipulation_description/urdf/turtlebot3_manipulation_robot.urdf.xacro (robot description, xacro)
@@ -11,3 +11,25 @@
     <child link="link1"/>
   </joint>
+  <link name="head_camera_link">
+    <inertial>
+      <mass value="0.1"/>
+      <origin xyz="0 0 0"/>
+      <inertia ixx="0.01" iyy="0.01" izz="0.01" ixy="0" ixz="0" iyz="0"/>
+    </inertial>
+    <collision>
+      <geometry>
+        <box size="0.05 0.05 0.05"/>
+      </geometry>
+    </collision>
+    <visual>
+      <geometry>
+        <box size="0.05 0.05 0.05"/>
+      </geometry>
+    </visual>
+  </link>
+  <joint name="head_camera_base_fixed" type="fixed">
+    <origin xyz="-0.3 0.3 0.6" rpy="0.0 0.6 -0.3"/>
+    <parent link="base_link"/>
+    <child link="head_camera_link"/>
+  </joint>
 </robot>

Commit message: add ros config

File: mechlmm_noetic_ws/src/turtlebot3_manipulation/turtlebot3_manipulation_description/urdf/open_manipulator_x.gazebo.xacro (robot description, xacro)
@@ -51,5 +51,5 @@
   <!-- camera -->
   <gazebo reference="hand_camera_link">
-    <sensor name="test_camera" type="depth">
+    <sensor name="hand_camera" type="depth">
       <update_rate>20</update_rate>
       <camera>
@@ -65,14 +65,14 @@
         </clip>
       </camera>
-      <plugin name="test_controller" filename="libgazebo_ros_openni_kinect.so">
+      <plugin name="hand_camera_controller" filename="libgazebo_ros_openni_kinect.so">
         <baseline>0.2</baseline>
         <alwaysOn>true</alwaysOn>
         <updateRate>1.0</updateRate>
-        <cameraName>test_ir</cameraName>
-        <imageTopicName>/test/color/image_raw</imageTopicName>
-        <cameraInfoTopicName>/test/color/camera_info</cameraInfoTopicName>
-        <depthImageTopicName>/test/depth/image_raw</depthImageTopicName>
-        <depthImageInfoTopicName>/test/depth/camera_info</depthImageInfoTopicName>
-        <pointCloudTopicName>/test/depth/points</pointCloudTopicName>
+        <cameraName>hand_camera_ir</cameraName>
+        <imageTopicName>/camera/hand/color/image_raw</imageTopicName>
+        <cameraInfoTopicName>/camera/hand/color/camera_info</cameraInfoTopicName>
+        <depthImageTopicName>/camera/hand/depth/image_raw</depthImageTopicName>
+        <depthImageInfoTopicName>/camera/hand/depth/camera_info</depthImageInfoTopicName>
+        <pointCloudTopicName>/camera/hand/depth/points</pointCloudTopicName>
         <frameName>hand_camera_link</frameName>
         <pointCloudCutoff>0.5</pointCloudCutoff>

File: mechlmm_noetic_ws/src/turtlebot3_manipulation/turtlebot3_manipulation_description/urdf/open_manipulator_x.urdf.xacro (robot description, xacro)
@@ -249,9 +249,9 @@
       </geometry>
     </visual> -->
-    <inertial>
+    <!-- <inertial>
       <mass value="0.1"/>
       <origin xyz="0 0 0"/>
       <inertia ixx="0.01" iyy="0.01" izz="0.01" ixy="0" ixz="0" iyz="0"/>
-    </inertial>
+    </inertial> -->
   </link>
   <joint name="hand_camera_base_fixed" type="fixed">
